File: pico_pad.kicad_pcb (KiCad board)
At the start: 2 copper layers, 95 x 95 mm, 26 parts, among them J1 Conn_01x20_Pin, J2 Conn_01x20_Pin, J3 Conn_01x10_Pin, J4 Conn_01x10_Pin, SW1 SW_Push, SW10 SW_Push, SW11 SW_Push, SW2 SW_Push, SW3 SW_Push, SW4 SW_Push, SW5 SW_Push, SW6 SW_Push, SW7 SW_Push, SW8 SW_Push, SW9 SW_Push

Commit message: update pcb
Parts:
- added RGB1: WS2812B, LED_SMD:LED_WS2812B-2020_PLCC4_2.0x2.0mm, B.Cu at (106.1, 59.4)
- added RGB10: WS2812B, LED_SMD:LED_WS2812B-2020_PLCC4_2.0x2.0mm, B.Cu at (115.6, 116.5)
- added RGB11: WS2812B, LED_SMD:LED_WS2812B-2020_PLCC4_2.0x2.0mm, B.Cu at (144.2, 116.5)
- added RGB2: WS2812B, LED_SMD:LED_WS2812B-2020_PLCC4_2.0x2.0mm, B.Cu at (125.2, 59.4)
- added RGB3: WS2812B, LED_SMD:LED_WS2812B-2020_PLCC4_2.0x2.0mm, B.Cu at (144.2, 59.4)
- added RGB4: WS2812B, LED_SMD:LED_WS2812B-2020_PLCC4_2.0x2.0mm, B.Cu at (106.1, 78.4)
- added RGB5: WS2812B, LED_SMD:LED_WS2812B-2020_PLCC4_2.0x2.0mm, B.Cu at (125.2, 78.4)
- added RGB6: WS2812B, LED_SMD:LED_WS2812B-2020_PLCC4_2.0x2.0mm, B.Cu at (144.2, 78.4)
- added RGB7: WS2812B, LED_SMD:LED_WS2812B-2020_PLCC4_2.0x2.0mm, B.Cu at (106.1, 97.5)
- added RGB8: WS2812B, LED_SMD:LED_WS2812B-2020_PLCC4_2.0x2.0mm, B.Cu at (125.2, 97.5)
- added RGB9: WS2812B, LED_SMD:LED_WS2812B-2020_PLCC4_2.0x2.0mm, B.Cu at (144.2, 97.5)
Routing:
- net (no net): track 0.00 -> 200.0 mm
- net COL0: track 179.9 -> 100.5 mm
- net COL1: track 163.8 -> 125.7 mm
- net COL2: track 153.8 -> 115.7 mm
- net ROW3: track 93.5 -> 88.5 mm
- net Net-(D8-A): track 6.57 -> 8.11 mm
- net Net-(D7-A): track 6.57 -> 8.11 mm
- net Net-(D5-A): track 6.57 -> 8.11 mm
- net Net-(D4-A): track 6.57 -> 8.11 mm
- net Net-(D2-A): track 6.57 -> 8.11 mm
- net Net-(D1-A): track 6.57 -> 8.11 mm
- net Net-(D9-A): track 6.57 -> 8.11 mm
- net Net-(D6-A): track 6.57 -> 8.11 mm
- net Net-(D3-A): track 6.57 -> 8.11 mm
- net Net-(D10-A): track 6.57 -> 8.11 mm
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
Commit message: update
Parts:
- D1, D10, D11, D2, D3, D4, D5, D6, D7, D8, D9: footprint Diode_SMD:D_SOD-323 -> Diode_SMD:D_SOD-123
- moved D11 3.00 mm to (149.4, 117.6)
- moved D1 3.00 mm to (111.2, 60.4)
- moved D10 3.00 mm to (120.7, 117.6)
- moved D2 3.00 mm to (130.3, 60.4)
- moved D3 3.00 mm to (149.3, 60.4)
- moved D4 3.00 mm to (111.2, 79.5)
- moved D5 3.00 mm to (130.3, 79.5)
- moved D6 3.00 mm to (149.3, 79.5)
- moved D7 3.00 mm to (111.2, 98.5)
- moved D8 3.00 mm to (130.3, 98.5)
- moved D9 3.00 mm to (149.3, 98.5)
Routing:
- net (no net): track 200.0 -> 57.1 mm
- net COL0: track 100.5 -> 185.2 mm
- net COL1: track 125.7 -> 167.3 mm
- net COL2: track 115.7 -> 153.8 mm
- net ROW3: track 88.5 -> 97.2 mm
- net ROW0: track 54.1 -> 58.2 mm
- net ROW1: track 70.6 -> 74.2 mm
- net ROW2: track 86.8 -> 90.4 mm
- net Net-(D11-A): track 8.11 -> 10.5 mm
- net Net-(D8-A): track 8.11 -> 10.5 mm
- net Net-(D7-A): track 8.11 -> 10.5 mm
- net Net-(D6-A): track 8.11 -> 10.5 mm
- net Net-(D5-A): track 8.11 -> 10.5 mm
- net Net-(D4-A): track 8.11 -> 10.5 mm
- net Net-(D10-A): track 8.11 -> 10.5 mm
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Other:
- board text added: "VBUS"
- board text removed: "locked"

Commit message: update pcb, add ws2812
Parts:
- RGB1, RGB10, RGB11, RGB2, RGB3, RGB4, RGB5, RGB6, RGB7, RGB8, RGB9: footprint LED_SMD:LED_WS2812B-2020_PLCC4_2.0x2.0mm -> LED_SMD:LED-SMD_L3.2-W2.8-BR_DY-S352818
